File: ACM - Align CAN-bus Module/AR19.MCU board/MCU board ATmega328p v2.3.sch (EAGLE design)
At the start: 36 parts, among them IC1 ATMEGA328P-MMH, IC2 MIC5239-5.0YS_TR, IC3 MCP25625-E_ML, J1 AVR_SPI_PROG_3X2NS

Commit message: Oppdatering MCP-25625
Parts:
- added C10, C9: 22pF, 12066D106KAT2A:12066D106KAT2A
- added QF2: 16M20AUM1, crystal:16M20AUM1
Connections:
- removed net N$7: IC1.PD2_(INT0/PCINT18)
- removed net OSC1: C2.2, IC1.(PCINT6/XTAL1/TOSC1)_PB6, IC3.OSC1, QF1.1
- removed net OSC2: C3.2, IC1.(PCINT7/XTAL2/TOSC2)_PB7, IC3.OSC2, QF1.3
- new net CAN_OSC1: C9.2, IC3.OSC1, QF2.1
- new net CAN_OSC2: C10.2, IC3.OSC2, QF2.3
- new net MCU_OSC1: C2.2, IC1.(PCINT6/XTAL1/TOSC1)_PB6, QF1.1
- new net MCU_OSC2: C3.2, IC1.(PCINT7/XTAL2/TOSC2)_PB7, QF1.3
- net CAN_INIT: now also IC1.PD2_(INT0/PCINT18)
- net GND: now also C10.1, C9.1, QF2.2
Other:
- moved on the sheet: C1, C4, IC2, R1, RES_PAD1, RES_PAD2
