File: ACM - Align CAN-bus Module/AR19.MCU board/MCU board ATmega328p v2.3.brd (EAGLE design)
At the start: 19 x 26.3 mm, 37 parts, among them IC1 ATMEGA328P-MMH, IC2 MIC5239-5.0YS_TR, IC3 MCP25625-E_ML, J1 AVR_SPI_PROG_3X2NS

Commit message: Created BOM 031018
Parts:
- added U$1, U$2: FA-20H, FA-20H 16.0000MF20X-B:FA-20H
Connections:
- net CAN_OSC1: now also U$1.1
- net CAN_OSC2: now also U$1.3
- net MCU_OSC1: now also U$2.1
- net MCU_OSC2: now also U$2.3
Changed lines of the file:
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@@
 <attribute name="VALUE" x="-5.715" y="-43.18" size="1.27" layer="27" align="center"/>
 </element>
+<element name="U$1" library="FA-20H 16.0000MF20X-B" package="FA-20H" value="FA-20H" x="-8.89" y="-52.705" smashed="yes"/>
+<element name="U$2" library="FA-20H 16.0000MF20X-B" package="FA-20H" value="FA-20H" x="-8.89" y="-57.15" smashed="yes"/>
 </elements>
 <signals>
@@
 <contactref element="IC1" pad="5"/>
 <contactref element="C2" pad="2"/>
-<wire x1="11.285" y1="10.98" x2="11.935" y2="21.59" width="0" layer="19" extent="1-1"/>
+<contactref element="U$2" pad="1"/>
+<wire x1="11.285" y1="10.98" x2="-8.09" y2="-56.4" width="0" layer="19" extent="1-1"/>
+<wire x1="11.935" y1="21.59" x2="11.285" y2="10.98" width="0" layer="19" extent="1-1"/>
 </signal>
 <signal name="MCU_OSC2">
 <contactref element="IC1" pad="6"/>
 <contactref element="C3" pad="2"/>
-<wire x1="11.285" y1="10.53" x2="14.735" y2="24.13" width="0" layer="19" extent="1-1"/>
+<contactref element="U$2" pad="3"/>
+<wire x1="11.285" y1="10.53" x2="-6.39" y2="-55" width="0" layer="19" extent="1-1"/>
+<wire x1="14.735" y1="24.13" x2="11.285" y2="10.53" width="0" layer="19" extent="1-1"/>
 </signal>
 <signal name="CAN_OSC1">
 <contactref element="IC3" pad="21"/>
 <contactref element="C9" pad="2"/>
+<contactref element="U$1" pad="1"/>
+<wire x1="-5.585" y1="-48.26" x2="-8.09" y2="-51.955" width="0" layer="19" extent="1-1"/>
 <wire x1="7.93" y1="15.92" x2="-5.585" y2="-48.26" width="0" layer="19" extent="1-1"/>
 </signal>
@@
 <contactref element="IC3" pad="20"/>
 <contactref element="C10" pad="2"/>
+<contactref element="U$1" pad="3"/>
+<wire x1="-0.505" y1="-48.26" x2="-6.39" y2="-50.555" width="0" layer="19" extent="1-1"/>
 <wire x1="7.93" y1="15.27" x2="-0.505" y2="-48.26" width="0" layer="19" extent="1-1"/>
 </signal>
