File: ACM - Align CAN-bus Module/AR19.MCU board/MCU board ATmega328p v2.4 (AW).brd (EAGLE design)
At the start: 160 x 100 mm, 49 parts, among them IC1 ATMEGA328P-MMH, IC2 MIC5239-5.0YS_TR, IC3 MCP25625-E_ML, J1 AVR_SPI_PROG_3X2NS, U1 CSTNE16M0V530000R0, U2 CSTNE16M0V530000R0

Commit message: Gotta stage it all - pokemon!
Parts:
- removed I/O_AD0: I/O_AD0, wirepad:2,15/1,0
- removed I/O_AD1: I/O_AD1, wirepad:2,15/1,0
- removed I/O_ADC2_SDA: I/O_ADC2_SDA, wirepad:2,15/1,0
- removed I/O_ADC3_SCL: I/O_ADC3_SCL, wirepad:2,15/1,0
- removed IC2: MIC5239-5.0YS_TR, MIC5239-5.0YS_TR:SOT230P700X170-4N
- added AD0: AD0, wirepad:2,15/1,0
- added AD1: AD1, wirepad:2,15/1,0
- added ADC2_SDA: ADC2_SDA, wirepad:2,15/1,0
- added ADC3_SCL: ADC3_SCL, wirepad:2,15/1,0
- added GND32: GND, wirepad:2,15/1,0
- added LDO: MIC5239-5.0YS_TR, MIC5239-5.0YS_TR:SOT230P700X170-4N
- PWM1_INT1: value PWM0_INT -> PWM1
- moved R8 234.1 mm to (31.9, 15.5), turned to 270 degrees
- moved R7 232.8 mm to (31.9, 18.5), turned to 270 degrees
- moved R6 231.6 mm to (31.9, 21.5), turned to 270 degrees
- moved R5 207.6 mm to (27.6, 6.20)
- moved R4 201.9 mm to (27.6, 2.05)
- moved R2 200.1 mm to (27.6, 4.15)
- moved LED1 194.9 mm to (26.8, 8.85), turned to 90 degrees
- moved U2 179.6 mm to (21.8, 2.55)
- moved C9 169.3 mm to (24.5, 2.54), turned to 270 degrees
- moved U1 164.7 mm to (11.8, 3.45), turned to 180 degrees
- moved C3 161.7 mm to (19.0, 2.54), turned to 270 degrees
- moved MOSI 156.3 mm to (37.5, 13.4)
- moved MISO 154.1 mm to (37.5, 15.9)
- moved SCK 152.1 mm to (37.5, 18.5)
- moved C2 150.6 mm to (9.10, 2.54), turned to 270 degrees
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Connections:
- net 12V_FUSED: now also LDO.1; no longer IC2.1
- net 5V: now also LDO.3; no longer IC2.3
- net GND: now also GND32.1, LDO.2, LDO.4; no longer IC2.2, IC2.4
- net N$3: now also AD1.1; no longer I/O_AD1.1
- net N$5: now also AD0.1; no longer I/O_AD0.1
- net N$6: now also ADC2_SDA.1; no longer I/O_ADC2_SDA.1
- net N$7: now also ADC3_SCL.1; no longer I/O_ADC3_SCL.1
Routing:
- net 5V: track 13.0 -> 62.6 mm, vias 2 -> 8
- net CAN_CS: track 0.00 -> 18.0 mm, vias 0 -> 2
- net MISO: track 0.00 -> 15.3 mm, vias 0 -> 3
- net SCK: track 0.00 -> 14.4 mm, vias 0 -> 3
- net CANL: track 0.00 -> 9.48 mm
- net RESET_MCU: track 0.00 -> 8.98 mm, vias 0 -> 2
- net CANH: track 0.00 -> 8.66 mm
- net N$8: track 0.00 -> 8.43 mm
- net N$3: track 0.00 -> 7.79 mm, vias 0 -> 2
- net N$9: track 0.00 -> 7.67 mm
- net VOLTAGE_CHECK: track 2.10 -> 9.75 mm, vias 0 -> 2
- net CAN_OSC2: track 0.00 -> 7.39 mm
- net RED_LED: track 0.00 -> 7.06 mm
- net N$5: track 0.00 -> 6.93 mm, vias 0 -> 2
- net TXCAN: track 0.00 -> 6.88 mm, vias 0 -> 2
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- added copper zone on layer 2, net 5V
- added copper zone on layer 1, net GND
Other:
- board size 160 x 100 mm -> 40 x 24 mm
