File: ACM - Align CAN-bus Module/AR19.MCU board/MCU board ATmega328p v2.4 (AW).sch (EAGLE design)
At the start: 49 parts, among them IC1 ATMEGA328P-MMH, IC2 MIC5239-5.0YS_TR, IC3 MCP25625-E_ML, J1 AVR_SPI_PROG_3X2NS, U1 CSTNE16M0V530000R0, U2 CSTNE16M0V530000R0

Commit message: Gotta stage it all - pokemon!
Parts:
- added GND32: GND, wirepad:2,15/1,0
- AD0: value I/O_AD0 -> AD0
- AD1: value I/O_AD1 -> AD1
- ADC2_SDA: value I/O_ADC2_SDA -> ADC2_SDA
- ADC3_SCL: value I/O_ADC3_SCL -> ADC3_SCL
- PWM1_INT1: value PWM0_INT -> PWM1
- renumbered I/O_AD0 to AD0, I/O_AD1 to AD1, I/O_ADC2_SDA to ADC2_SDA, I/O_ADC3_SCL to ADC3_SCL, IC2 to LDO
Connections:
- net GND: now also GND32.P
Changed lines of the file:
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@@
 <parts>
 <part name="IC1" library="ATMEGA328P-MMH" deviceset="ATMEGA328P-MMH" device=""/>
-<part name="IC2" library="MIC5239-5.0YS_TR" deviceset="MIC5239-5.0YS_TR" device=""/>
+<part name="LDO" library="MIC5239-5.0YS_TR" deviceset="MIC5239-5.0YS_TR" device=""/>
 <part name="IC3" library="MCP25625-E_ML" deviceset="MCP25625-E_ML" device=""/>
 <part name="J1" library="SparkFun-Connectors" deviceset="AVR_SPI_PROG_3X2" device="NS"/>
@@
 <part name="CANH" library="wirepad" library_urn="urn:adsk.eagle:library:412" deviceset="2,15/1,0" device="" package3d_urn="urn:adsk.eagle:package:30831/1" value="I/O_CANH"/>
 <part name="CANL" library="wirepad" library_urn="urn:adsk.eagle:library:412" deviceset="2,15/1,0" device="" package3d_urn="urn:adsk.eagle:package:30831/1" value="I/O_CANH"/>
-<part name="PWM1_INT1" library="wirepad" library_urn="urn:adsk.eagle:library:412" deviceset="2,15/1,0" device="" package3d_urn="urn:adsk.eagle:package:30831/1" value="PWM0_INT"/>
+<part name="PWM1_INT1" library="wirepad" library_urn="urn:adsk.eagle:library:412" deviceset="2,15/1,0" device="" package3d_urn="urn:adsk.eagle:package:30831/1" value="PWM1"/>
 <part name="C5" library="eagle-ltspice" library_urn="urn:adsk.eagle:library:217" deviceset="C" device="C0603" package3d_urn="urn:adsk.eagle:package:13262/1" value="22pF"/>
 <part name="C6" library="eagle-ltspice" library_urn="urn:adsk.eagle:library:217" deviceset="C" device="C0603" package3d_urn="urn:adsk.eagle:package:13262/1" value="0.1uF"/>
@@
 <part name="MISO" library="wirepad" library_urn="urn:adsk.eagle:library:412" deviceset="2,15/1,0" device="" package3d_urn="urn:adsk.eagle:package:30831/1" value="MISO"/>
 <part name="MOSI" library="wirepad" library_urn="urn:adsk.eagle:library:412" deviceset="2,15/1,0" device="" package3d_urn="urn:adsk.eagle:package:30831/1" value="MOSI"/>
-<part name="I/O_ADC3_SCL" library="wirepad" library_urn="urn:adsk.eagle:library:412" deviceset="2,15/1,0" device="" package3d_urn="urn:adsk.eagle:package:30831/1" value="I/O_ADC3_SCL"/>
-<part name="I/O_ADC2_SDA" library="wirepad" library_urn="urn:adsk.eagle:library:412" deviceset="2,15/1,0" device="" package3d_urn="urn:adsk.eagle:package:30831/1" value="I/O_ADC2_SDA"/>
-<part name="I/O_AD0" library="wirepad" library_urn="urn:adsk.eagle:library:412" deviceset="2,15/1,0" device="" package3d_urn="urn:adsk.eagle:package:30831/1" value="I/O_AD0"/>
+<part name="ADC3_SCL" library="wirepad" library_urn="urn:adsk.eagle:library:412" deviceset="2,15/1,0" device="" package3d_urn="urn:adsk.eagle:package:30831/1" value="ADC3_SCL"/>
+<part name="ADC2_SDA" library="wirepad" library_urn="urn:adsk.eagle:library:412" deviceset="2,15/1,0" device="" package3d_urn="urn:adsk.eagle:package:30831/1" value="ADC2_SDA"/>
+<part name="AD0" library="wirepad" library_urn="urn:adsk.eagle:library:412" deviceset="2,15/1,0" device="" package3d_urn="urn:adsk.eagle:package:30831/1" value="AD0"/>
 <part name="C2" library="eagle-ltspice" library_urn="urn:adsk.eagle:library:217" deviceset="C" device="C0603" package3d_urn="urn:adsk.eagle:package:13262/1" value="22pF"/>
 <part name="C3" library="eagle-ltspice" library_urn="urn:adsk.eagle:library:217" deviceset="C" device="C0603" package3d_urn="urn:adsk.eagle:package:13262/1" value="22pF"/>
@@
 <part name="SUPPLY15" library="SparkFun-PowerSymbols" deviceset="5V" device=""/>
 <part name="PWM0" library="wirepad" library_urn="urn:adsk.eagle:library:412" deviceset="2,15/1,0" device="" package3d_urn="urn:adsk.eagle:package:30831/1" value="PWM0"/>
-<part name="I/O_AD1" library="wirepad" library_urn="urn:adsk.eagle:library:412" deviceset="2,15/1,0" device="" package3d_urn="urn:adsk.eagle:package:30831/1" value="I/O_AD1"/>
+<part name="AD1" library="wirepad" library_urn="urn:adsk.eagle:library:412" deviceset="2,15/1,0" device="" package3d_urn="urn:adsk.eagle:package:30831/1" value="AD1"/>
 <part name="R6" library="eagle-ltspice" library_urn="urn:adsk.eagle:library:217" deviceset="R" device="R0603" package3d_urn="urn:adsk.eagle:package:13302/1" value="200Ohm"/>
 <part name="R7" library="eagle-ltspice" library_urn="urn:adsk.eagle:library:217" deviceset="R" device="R0603" package3d_urn="urn:adsk.eagle:package:13302/1" value="200Ohm"/>
@@
 <part name="5V" library="wirepad" library_urn="urn:adsk.eagle:library:412" deviceset="2,15/1,0" device="" package3d_urn="urn:adsk.eagle:package:30831/1" value="5V"/>
 <part name="SUPPLY3" library="SparkFun-PowerSymbols" deviceset="5V" device=""/>
+<part name="GND32" library="wirepad" library_urn="urn:adsk.eagle:library:412" deviceset="2,15/1,0" device="" package3d_urn="urn:adsk.eagle:package:30831/1" value="GND"/>
+<part name="GND33" library="supply1" library_urn="urn:adsk.eagle:library:371" deviceset="GND" device=""/>
 </parts>
 <sheets>
@@
 <attribute name="VALUE" x="31.75" y="86.36" size="1.778" layer="96" align="center-left"/>
 </instance>
-<instance part="IC2" gate="G$1" x="-17.78" y="162.56">
+<instance part="LDO" gate="G$1" x="-17.78" y="162.56">
 <attribute name="NAME" x="-13.97" y="167.64" size="1.778" layer="95" align="center-left"/>
 <attribute name="VALUE" x="-13.97" y="170.18" size="1.778" layer="96" align="center-left"/>
@@
 <attribute name="VALUE" x="108.077" y="-87.122" size="1.778" layer="96"/>
 </instance>
-<instance part="I/O_ADC3_SCL" gate="1" x="91.44" y="63.5" rot="R180">
+<instance part="ADC3_SCL" gate="1" x="91.44" y="63.5" rot="R180">
 <attribute name="NAME" x="92.837" y="62.8142" size="1.778" layer="95"/>
 </instance>
-<instance part="I/O_ADC2_SDA" gate="1" x="91.44" y="58.42" rot="R180">
+<instance part="ADC2_SDA" gate="1" x="91.44" y="58.42" rot="R180">
 <attribute name="NAME" x="92.837" y="57.7342" size="1.778" layer="95"/>
 </instance>
-<instance part="I/O_AD0" gate="1" x="91.44" y="53.34" rot="R180">
+<instance part="AD0" gate="1" x="91.44" y="53.34" rot="R180">
 <attribute name="NAME" x="92.837" y="52.6542" size="1.778" layer="95"/>
 </instance>
@@
 <attribute name="NAME" x="18.923" y="-71.8058" size="1.778" layer="95" rot="MR0"/>
 </instance>
-<instance part="I/O_AD1" gate="1" x="91.44" y="48.26" rot="R180">
+<instance part="AD1" gate="1" x="91.44" y="48.26" rot="R180">
 <attribute name="VALUE" x="92.837" y="47.498" size="1.778" layer="96"/>
 </instance>
@@
 <instance part="SUPPLY3" gate="G$1" x="-58.42" y="144.78" rot="R180">
 <attribute name="VALUE" x="-58.42" y="141.986" size="1.778" layer="96" rot="R180" align="bottom-center"/>
+</instance>
+<instance part="GND32" gate="1" x="-81.28" y="149.86" rot="R270">
+<attribute name="VALUE" x="-84.582" y="151.003" size="1.778" layer="96" rot="R270"/>
+</instance>
+<instance part="GND33" gate="1" x="-81.28" y="142.24" rot="MR0">
+<attribute name="VALUE" x="-78.74" y="139.7" size="1.778" layer="96" rot="MR0"/>
 </instance>
 </instances>
@@
 </segment>
 <segment>
-<pinref part="IC2" gate="G$1" pin="OUT"/>
+<pinref part="LDO" gate="G$1" pin="OUT"/>
 <wire x1="7.62" y1="162.56" x2="17.78" y2="162.56" width="0.1524" layer="91"/>
 <pinref part="SUPPLY2" gate="G$1" pin="5V"/>
@@
 <segment>
 <pinref part="GND2" gate="1" pin="GND"/>
-<pinref part="IC2" gate="G$1" pin="GND"/>
+<pinref part="LDO" gate="G$1" pin="GND"/>
 <wire x1="-17.78" y1="160.02" x2="-22.86" y2="160.02" width="0.1524" layer="91"/>
 <wire x1="-22.86" y1="160.02" x2="-22.86" y2="144.78" width="0.1524" layer="91"/>
@@
 </segment>
 <segment>
-<pinref part="IC2" gate="G$1" pin="TAB"/>
+<pinref part="LDO" gate="G$1" pin="TAB"/>
 <wire x1="7.62" y1="160.02" x2="10.16" y2="160.02" width="0.1524" layer="91"/>
 <pinref part="GND12" gate="1" pin="GND"/>
@@
 <pinref part="GND31" gate="1" pin="GND"/>
 <wire x1="-66.04" y1="147.32" x2="-66.04" y2="144.78" width="0.1524" layer="91"/>
+</segment>
+<segment>
+<pinref part="GND32" gate="1" pin="P"/>
+<pinref part="GND33" gate="1" pin="GND"/>
+<wire x1="-81.28" y1="147.32" x2="-81.28" y2="144.78" width="0.1524" layer="91"/>
 </segment>
 </net>
@@
 <pinref part="FUSE" gate="G$1" pin="2"/>
 <wire x1="-43.18" y1="162.56" x2="-33.02" y2="162.56" width="0.1524" layer="91"/>
-<pinref part="IC2" gate="G$1" pin="IN"/>
+<pinref part="LDO" gate="G$1" pin="IN"/>
 <wire x1="-33.02" y1="162.56" x2="-33.02" y2="160.02" width="0.1524" layer="91"/>
 <wire x1="-17.78" y1="162.56" x2="-33.02" y2="162.56" width="0.1524" layer="91"/>
@@
 <wire x1="48.26" y1="50.8" x2="48.26" y2="53.34" width="0.1524" layer="91"/>
 <wire x1="48.26" y1="53.34" x2="88.9" y2="53.34" width="0.1524" layer="91"/>
-<pinref part="I/O_AD0" gate="1" pin="P"/>
+<pinref part="AD0" gate="1" pin="P"/>
 </segment>
 </net>
@@
 <wire x1="45.72" y1="50.8" x2="45.72" y2="58.42" width="0.1524" layer="91"/>
 <wire x1="45.72" y1="58.42" x2="88.9" y2="58.42" width="0.1524" layer="91"/>
-<pinref part="I/O_ADC2_SDA" gate="1" pin="P"/>
+<pinref part="ADC2_SDA" gate="1" pin="P"/>
 </segment>
 </net>
@@
 <wire x1="43.18" y1="50.8" x2="43.18" y2="63.5" width="0.1524" layer="91"/>
 <wire x1="43.18" y1="63.5" x2="88.9" y2="63.5" width="0.1524" layer="91"/>
-<pinref part="I/O_ADC3_SCL" gate="1" pin="P"/>
+<pinref part="ADC3_SCL" gate="1" pin="P"/>
 </segment>
 </net>
@@
 <wire x1="81.28" y1="12.7" x2="81.28" y2="48.26" width="0.1524" layer="91"/>
 <wire x1="81.28" y1="48.26" x2="88.9" y2="48.26" width="0.1524" layer="91"/>
-<pinref part="I/O_AD1" gate="1" pin="P"/>
-</segment>
-</net>
+<pinref part="AD1" gate="1" pin="P"/>
+</segment>
+</net>
