File: Brakelight/PCB/Brakelight_v3/Brakelight_v3.sch (EAGLE design)
At the start: 57 parts, among them U1 LM358MX

Commit message: Brakelight only stubs left
Connections:
- net N$36 renamed LEDK
Changed lines of the file:
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@@
 </segment>
 </net>
-<net name="N$36" class="0">
+<net name="LEDK" class="0">
 <segment>
 <pinref part="LED51" gate="G$1" pin="K"/>
