File: Main ACM Hub/Main ACM Hub.brd (EAGLE design)
At the start: 259.1 x 129.5 mm, 10 parts

Commit message: Change: ACM_Hub
Parts:
- moved U$10 15.5 mm to (193.0, 15.2)
- moved U$2 15.5 mm to (15.2, 14.0)
- moved U$6 15.5 mm to (104.1, 14.0)
- moved U$9 15.5 mm to (193.0, 54.6)
- moved U$1 15.5 mm to (59.7, 14.0)
- moved U$5 15.5 mm to (148.6, 14.0)
- moved U$4 15.5 mm to (15.2, 54.6)
- moved U$8 15.5 mm to (104.1, 54.6)
- moved U$3 15.5 mm to (59.7, 54.6)
- moved U$7 15.5 mm to (148.6, 54.6)
Other:
- board size 259.1 x 129.5 mm -> 240 x 106.7 mm
Changed lines of the file:
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@@
 <?xml version="1.0" encoding="utf-8"?>
 <!DOCTYPE eagle SYSTEM "eagle.dtd">
-<eagle version="9.2.1">
+<eagle version="9.2.2">
 <drawing>
 <settings>
@@
 <board>
 <plain>
-<wire x1="0" y1="0" x2="259.06" y2="0" width="0" layer="20"/>
-<wire x1="259.06" y1="0" x2="259.07" y2="129.54" width="0" layer="20"/>
-<wire x1="259.07" y1="129.54" x2="0.01" y2="129.54" width="0" layer="20"/>
-<wire x1="0.01" y1="129.54" x2="0" y2="0" width="0" layer="20"/>
+<wire x1="0" y1="0" x2="240.01" y2="0" width="0" layer="20"/>
+<wire x1="240.01" y1="0" x2="240.02" y2="106.68" width="0" layer="20"/>
+<wire x1="240.02" y1="106.68" x2="0.01" y2="106.68" width="0" layer="20"/>
+<wire x1="0.01" y1="106.68" x2="0" y2="0" width="0" layer="20"/>
+<dimension x1="0" y1="0" x2="0" y2="14.986" x3="-4.191" y3="7.493" textsize="1.778" layer="1"/>
 </plain>
 <attributes>
@@
 </autorouter>
 <elements>
-<element name="U$1" library="ACM_Pindown" package="ACM_CAS_FP" value="ACM_CASTELLATED" x="62.23" y="29.21" smashed="yes"/>
-<element name="U$10" library="ACM_Pindown" package="ACM_CAS_FP" value="ACM_CASTELLATED" x="195.58" y="30.48" smashed="yes"/>
-<element name="U$2" library="ACM_Pindown" package="ACM_CAS_FP" value="ACM_CASTELLATED" x="17.78" y="29.21" smashed="yes"/>
-<element name="U$3" library="ACM_Pindown" package="ACM_CAS_FP" value="ACM_CASTELLATED" x="62.23" y="69.85" smashed="yes"/>
-<element name="U$4" library="ACM_Pindown" package="ACM_CAS_FP" value="ACM_CASTELLATED" x="17.78" y="69.85" smashed="yes"/>
-<element name="U$5" library="ACM_Pindown" package="ACM_CAS_FP" value="ACM_CASTELLATED" x="151.13" y="29.21" smashed="yes"/>
-<element name="U$6" library="ACM_Pindown" package="ACM_CAS_FP" value="ACM_CASTELLATED" x="106.68" y="29.21" smashed="yes"/>
-<element name="U$7" library="ACM_Pindown" package="ACM_CAS_FP" value="ACM_CASTELLATED" x="151.13" y="69.85" smashed="yes"/>
-<element name="U$8" library="ACM_Pindown" package="ACM_CAS_FP" value="ACM_CASTELLATED" x="106.68" y="69.85" smashed="yes"/>
-<element name="U$9" library="ACM_Pindown" package="ACM_CAS_FP" value="ACM_CASTELLATED" x="195.58" y="69.85" smashed="yes"/>
+<element name="U$1" library="ACM_Pindown" package="ACM_CAS_FP" value="ACM_CASTELLATED" x="59.69" y="13.97" smashed="yes"/>
+<element name="U$10" library="ACM_Pindown" package="ACM_CAS_FP" value="ACM_CASTELLATED" x="193.04" y="15.24" smashed="yes"/>
+<element name="U$2" library="ACM_Pindown" package="ACM_CAS_FP" value="ACM_CASTELLATED" x="15.24" y="13.97" smashed="yes"/>
+<element name="U$3" library="ACM_Pindown" package="ACM_CAS_FP" value="ACM_CASTELLATED" x="59.69" y="54.61" smashed="yes"/>
+<element name="U$4" library="ACM_Pindown" package="ACM_CAS_FP" value="ACM_CASTELLATED" x="15.24" y="54.61" smashed="yes"/>
+<element name="U$5" library="ACM_Pindown" package="ACM_CAS_FP" value="ACM_CASTELLATED" x="148.59" y="13.97" smashed="yes"/>
+<element name="U$6" library="ACM_Pindown" package="ACM_CAS_FP" value="ACM_CASTELLATED" x="104.14" y="13.97" smashed="yes"/>
+<element name="U$7" library="ACM_Pindown" package="ACM_CAS_FP" value="ACM_CASTELLATED" x="148.59" y="54.61" smashed="yes"/>
+<element name="U$8" library="ACM_Pindown" package="ACM_CAS_FP" value="ACM_CASTELLATED" x="104.14" y="54.61" smashed="yes"/>
+<element name="U$9" library="ACM_Pindown" package="ACM_CAS_FP" value="ACM_CASTELLATED" x="193.04" y="54.61" smashed="yes"/>
 </elements>
 <signals>
