File: ACM_Hotswap board/PCB/ACM_HotswapMultiboard.sch (EAGLE design)
At the start: 19 parts, among them IC1 Optocoupler DIP, Q1 NGD8201ANT4G, Q2 NGD8201ANT4G

Commit message: ACM_Hub_Progress 2
Parts:
- removed MOS0, MOS1: (no value), wirepad:2,15/1,0
- added U$5: 16P_CONNECTOR, 4P_Connector holes:16P_CONNECTOR
- U$3, U$4: device 4P_Connector holes - Copy:16P_CONNECTOR -> 4P_Connector holes:16P_CONNECTOR
Connections:
- removed net N$1: MOS0.P, R3.2
- removed net N$10: U$2.P$1
- removed net N$11: U$2.P$2
- removed net N$12: U$2.P$3
- removed net N$14: U$2.P$4
- removed net N$15: U$2.P$5
- removed net N$16: U$2.P$6
- removed net N$17: U$2.P$9
- removed net N$18: U$2.P$10
- removed net N$19: U$2.P$11
- removed net N$20: U$2.P$12
- removed net N$21: U$2.P$13
- removed net N$22: U$2.P$14
- removed net N$3: MOS1.P, R4.2
- net 12V: now also U$3.1, U$4.2, U$5.3; no longer U$3.12V, U$4.12V
- net 5V: now also U$2.2
- net 5V1: now also U$2.1
- net AD0: now also U$2.12
- net AD1: now also U$2.11
- net AD2: now also U$2.10
- net AD3: now also U$2.9
- net CANH: now also U$3.2, U$4.1, U$5.4; no longer U$3.CANH, U$4.CANH
- net CANL: now also U$3.3, U$4.4, U$5.1; no longer U$3.CANL, U$4.CANL
- net GND: now also U$2.3, U$3.4, U$4.3, U$5.2; no longer U$3.GND, U$4.GND
- net MISO: now also U$2.8
- net MOSI: now also U$2.7
- net PWM0: now also R3.2, U$2.4
- net PWM1: now also R4.2, U$2.5
- net SCK: now also U$2.6

Commit message: ACM_Hub (Hotswap) Ready
Connections:
- removed net 5V1: U$1.5V1, U$2.1
- net 5V: now also U$1.5V1, U$2.4, U$2.5; no longer U$2.2
- net PWM0: now also U$2.1; no longer U$2.4
- net PWM1: now also U$2.2; no longer U$2.5
Changed lines of the file:
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@@
 </segment>
 <segment>
-<pinref part="U$2" gate="G$1" pin="2"/>
-<wire x1="10.16" y1="78.74" x2="0" y2="78.74" width="0.1524" layer="91"/>
-<label x="0" y="78.74" size="1.778" layer="95"/>
+<pinref part="U$1" gate="G$1" pin="5V1"/>
+<wire x1="50.8" y1="29.21" x2="70.358" y2="29.21" width="0.1524" layer="91"/>
+<label x="70.358" y="29.21" size="1.778" layer="95"/>
+</segment>
+<segment>
+<pinref part="U$2" gate="G$1" pin="5"/>
+<wire x1="10.16" y1="86.36" x2="0" y2="86.36" width="0.1524" layer="91"/>
+<label x="0" y="86.36" size="1.778" layer="95"/>
+</segment>
+<segment>
+<pinref part="U$2" gate="G$1" pin="4"/>
+<wire x1="10.16" y1="83.82" x2="0" y2="83.82" width="0.1524" layer="91"/>
+<label x="0" y="83.82" size="1.778" layer="95"/>
 </segment>
 </net>
@@
 </segment>
 <segment>
-<pinref part="U$2" gate="G$1" pin="4"/>
-<wire x1="10.16" y1="83.82" x2="0" y2="83.82" width="0.1524" layer="91"/>
-<label x="0" y="83.82" size="1.778" layer="95"/>
-</segment>
-<segment>
 <pinref part="R3" gate="G$1" pin="2"/>
 <wire x1="-27.94" y1="5.08" x2="-20.32" y2="5.08" width="0.1524" layer="91"/>
 <label x="-27.94" y="5.08" size="1.778" layer="95"/>
+</segment>
+<segment>
+<pinref part="U$2" gate="G$1" pin="1"/>
+<wire x1="10.16" y1="76.2" x2="0" y2="76.2" width="0.1524" layer="91"/>
+<label x="0" y="76.2" size="1.778" layer="95"/>
 </segment>
 </net>
@@
 </segment>
 <segment>
-<pinref part="U$2" gate="G$1" pin="5"/>
-<wire x1="10.16" y1="86.36" x2="0" y2="86.36" width="0.1524" layer="91"/>
-<label x="0" y="86.36" size="1.778" layer="95"/>
-</segment>
-<segment>
 <pinref part="R4" gate="G$1" pin="2"/>
 <wire x1="-27.94" y1="0" x2="-20.574" y2="0" width="0.1524" layer="91"/>
 <label x="-27.94" y="0" size="1.778" layer="95"/>
+</segment>
+<segment>
+<pinref part="U$2" gate="G$1" pin="2"/>
+<wire x1="10.16" y1="78.74" x2="0" y2="78.74" width="0.1524" layer="91"/>
+<label x="0" y="78.74" size="1.778" layer="95"/>
 </segment>
 </net>
@@
 </segment>
 </net>
-<net name="5V1" class="0">
-<segment>
-<pinref part="U$1" gate="G$1" pin="5V1"/>
-<wire x1="50.8" y1="29.21" x2="70.358" y2="29.21" width="0.1524" layer="91"/>
-<label x="70.358" y="29.21" size="1.778" layer="95"/>
-</segment>
-<segment>
-<pinref part="U$2" gate="G$1" pin="1"/>
-<wire x1="10.16" y1="76.2" x2="0" y2="76.2" width="0.1524" layer="91"/>
-<label x="0" y="76.2" size="1.778" layer="95"/>
-</segment>
-</net>
