File: ACM_Hotswap board/PCB/ACM_HotswapMultiboard.brd (EAGLE design)
At the start: 50 x 50 mm, 19 parts, among them IC1 Optocoupler DIP

Commit message: ACM_Hub_Progress 2
Parts:
- removed MOS0, MOS1: (no value), wirepad:2,15/1,0
- added U$5: 16P_CONNECTOR, 4P_Connector holes:16P_CONNECTOR_FP
- U$3, U$4: device 4P_Connector holes - Copy:16P_CONNECTOR_FP -> 4P_Connector holes:16P_CONNECTOR_FP
- moved D0 44.3 mm to (47.9, 10.9), turned to 270 degrees
- moved D1 37.6 mm to (48.1, 22.4), turned to 90 degrees
- moved R4 30.1 mm to (12.8, 10.7)
- moved R3 28.3 mm to (16.0, 10.7)
- moved IC1 23.1 mm to (22.4, 7.54), turned to 180 degrees
- moved R5 21.4 mm to (28.6, 3.82), turned to 180 degrees
- moved Q1 18.0 mm to (33.0, 8.06), turned to 270 degrees
- moved U$2 17.5 mm to (18.7, 30.9)
- moved U$1 17.3 mm to (9.00, 2.00)
- moved U$4 15.7 mm to (46.0, 34.0)
- moved S1 15.4 mm to (48.1, 26.4)
- moved U$3 14.0 mm to (3.00, 34.0)
- moved R7 13.6 mm to (28.4, 10.4), turned to 90 degrees
- moved S0 12.1 mm to (48.1, 14.9)
- moved R2 10.8 mm to (32.0, 14.6), turned to 180 degrees
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Connections:
- removed net N$1: MOS0.1, R3.2
- removed net N$10: U$2.P$1
- removed net N$11: U$2.P$2
- removed net N$12: U$2.P$3
- removed net N$14: U$2.P$4
- removed net N$15: U$2.P$5
- removed net N$16: U$2.P$6
- removed net N$17: U$2.P$9
- removed net N$18: U$2.P$10
- removed net N$19: U$2.P$11
- removed net N$20: U$2.P$12
- removed net N$21: U$2.P$13
- removed net N$22: U$2.P$14
- removed net N$3: MOS1.1, R4.2
- net 12V: now also U$3.1, U$4.2, U$5.3; no longer U$3.12V, U$4.12V
- net 5V: now also U$2.2
- net 5V1: now also U$2.1
- net AD0: now also U$2.12
- net AD1: now also U$2.11
- net AD2: now also U$2.10
- net AD3: now also U$2.9
- net CANH: now also U$3.2, U$4.1, U$5.4; no longer U$3.CANH, U$4.CANH
- net CANL: now also U$3.3, U$4.4, U$5.1; no longer U$3.CANL, U$4.CANL
- net GND: now also U$2.3, U$3.4, U$4.3, U$5.2; no longer U$3.GND, U$4.GND
- net MISO: now also U$2.8
- net MOSI: now also U$2.7
- net PWM0: now also R3.2, U$2.4
- net PWM1: now also R4.2, U$2.5
- net SCK: now also U$2.6
Routing:
- net 12V: track 9.27 -> 98.3 mm
- net CANL: track 0.00 -> 86.8 mm
- net CANH: track 0.00 -> 78.1 mm, vias 0 -> 3
- net DRAIN1: track 0.00 -> 47.0 mm
- net PWM1: track 0.00 -> 41.6 mm
- net PWM0: track 0.00 -> 40.7 mm
- net MOSI: track 0.00 -> 33.3 mm
- net SCK: track 0.00 -> 32.7 mm
- net GATE1: track 0.00 -> 32.2 mm
- net MISO: track 0.00 -> 29.5 mm
- net SOURCE1: track 0.00 -> 27.2 mm
- net AD3: track 0.00 -> 25.7 mm
- net AD2: track 0.00 -> 21.6 mm
- net AD1: track 0.00 -> 17.7 mm
- net AD0: track 0.00 -> 13.3 mm
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- removed copper zone on layer 16, net GND
Other:
- board size 50 x 50 mm -> 52 x 37 mm

Commit message: ACM_Hub (Hotswap) Ready
Parts:
- moved R7 2.06 mm to (28.1, 12.4)
- moved R5 1.00 mm to (28.6, 4.82)
- moved D0 1.00 mm to (47.9, 11.9)
- moved D1 1.00 mm to (48.1, 23.4)
- moved Q1 1.00 mm to (33.0, 9.06)
- moved Q2 1.00 mm to (25.0, 24.1)
- moved R1 1.00 mm to (31.7, 25.4)
- moved R2 1.00 mm to (32.0, 15.6)
- moved R3 1.00 mm to (16.0, 11.7)
- moved R4 1.00 mm to (12.8, 11.7)
- moved S0 1.00 mm to (48.1, 15.9)
- moved S1 1.00 mm to (48.1, 27.4)
- moved U$1 1.00 mm to (9.00, 3.00)
- moved U$2 1.00 mm to (18.7, 31.9)
- moved U$3 1.00 mm to (3.00, 35.0)
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Connections:
- removed net 5V1: U$1.5V1_P, U$2.1
- net 5V: now also U$1.5V1_P, U$2.4, U$2.5; no longer U$2.2
- net PWM0: now also U$2.1; no longer U$2.4
- net PWM1: now also U$2.2; no longer U$2.5
Routing:
- net SOURCE0: track 0.00 -> 34.4 mm
- net DRAIN0: track 0.00 -> 29.3 mm
- net GATE0: track 0.00 -> 10.4 mm
- net PWM0: track 40.7 -> 30.4 mm
- net 12V: track 98.3 -> 88.9 mm
- net GND: track 0.00 -> 7.81 mm, vias 0 -> 2
- net PWM1: track 41.6 -> 34.5 mm
- net CANH: track 78.1 -> 80.9 mm, vias 3 -> 2
- net N$7: track 0.00 -> 1.60 mm
- net DRAIN1: track 47.0 -> 45.8 mm
- added copper zone on layer 1, net 5V
- added copper zone on layer 16, net GND
Other:
- board size 52 x 37 mm -> 52 x 38 mm

Commit message: ACM Hotswap ready for prduction
Routing:
- net GND: track 7.81 -> 10.6 mm, vias 2 -> 4
- net SOURCE1: track 27.2 -> 26.5 mm
- net CANL: track 86.8 -> 87.5 mm
- net SCK: track 32.7 -> 32.1 mm
Other:
- board text added: "12V"
- board text added: "AD0 | SCK"
- board text added: "AD1 | 5V"
- board text added: "AD2 | 5V"
- board text added: "AD3 | GND"
- board text added: "CANH"
- board text added: "CANL"
- board text added: "GND"
- board text added: "MISO | PWM1"
- board text added: "MOSI | PWM0"
Changed lines of the file:
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@@
 <setting verticaltext="up"/>
 </settings>
-<grid distance="1" unitdist="mm" unit="mm" style="lines" multiple="1" display="no" altdistance="0.01" altunitdist="mm" altunit="mm"/>
+<grid distance="1" unitdist="mm" unit="mm" style="lines" multiple="1" display="yes" altdistance="0.01" altunitdist="mm" altunit="mm"/>
 <layers>
 <layer number="1" name="Top" color="4" fill="1" visible="yes" active="yes"/>
@@
 <wire x1="0" y1="38" x2="0" y2="0" width="0" layer="20"/>
 <text x="46.36" y="6.53" size="4" layer="26" distance="0">+</text>
-<text x="47.17" y="16.53" size="4" layer="25" distance="0">-</text>
+<text x="47.17" y="16.53" size="4" layer="26" distance="0">-</text>
 <text x="46.41" y="18.36" size="4" layer="26" distance="0">+</text>
 <text x="47.39" y="28.11" size="4" layer="26" distance="0">-</text>
+<text x="1.94" y="36.18" size="1" layer="25">12V</text>
+<text x="4.76" y="36.12" size="1" layer="25">CANH</text>
+<text x="0.41" y="30.38" size="1" layer="25">CANL</text>
+<text x="4.57" y="30.38" size="1" layer="25">GND</text>
+<text x="1.86" y="0.49" size="1" layer="25">12V</text>
+<text x="4.62" y="0.4" size="1" layer="25">CANH</text>
+<text x="4.67" y="5.99" size="1" layer="25">GND</text>
+<text x="0.65" y="6.08" size="1" layer="25">CANL</text>
+<text x="43.15" y="36.06" size="1" layer="25">CANH</text>
+<text x="47.79" y="36.12" size="1" layer="25">12V</text>
+<text x="43.92" y="30.37" size="1" layer="25">GND</text>
+<text x="47.63" y="30.47" size="1" layer="25">CANL</text>
+<hole x="13" y="6" drill="2"/>
+<hole x="10" y="3" drill="3"/>
+<hole x="42" y="33" drill="3"/>
+<hole x="10" y="33" drill="3"/>
+<text x="19" y="33" size="0.5" layer="25" rot="R90">MOSI | PWM0</text>
+<text x="21.56" y="33" size="0.5" layer="25" rot="R90">MISO | PWM1</text>
+<text x="24.12" y="33" size="0.5" layer="25" rot="R90">AD3 | GND</text>
+<text x="26.68" y="33" size="0.5" layer="25" rot="R90">AD2 | 5V</text>
+<text x="29.24" y="33" size="0.5" layer="25" rot="R90">AD1 | 5V</text>
+<text x="31.8" y="33" size="0.5" layer="25" rot="R90">AD0 | SCK</text>
 </plain>
 <attributes>
@@
 <wire x1="12.38" y1="20.48" x2="14.62" y2="18.24" width="1" layer="1"/>
 <wire x1="14.62" y1="18.24" x2="14.81" y2="18.24" width="1" layer="1"/>
+<via x="6" y="8" extent="1-16" drill="1"/>
+<via x="6.66" y="10.48" extent="1-16" drill="1"/>
+<wire x1="6" y1="8" x2="6" y2="9.82" width="1" layer="1"/>
+<wire x1="6" y1="9.82" x2="6.66" y2="10.48" width="1" layer="1"/>
 </signal>
 <signal name="GATE1">
@@
 <wire x1="31.73" y1="22.73936875" x2="30.78523125" y2="21.7946" width="1" layer="16"/>
 <wire x1="29.18" y1="21.777" x2="32.00215625" y2="21.777" width="2" layer="16"/>
-<wire x1="32.00215625" y1="21.777" x2="38.91155625" y2="28.6864" width="2" layer="16"/>
-<wire x1="48.08" y1="27.406" x2="46.7996" y2="28.6864" width="2" layer="16"/>
-<wire x1="46.7996" y1="28.6864" x2="38.91155625" y2="28.6864" width="2" layer="16"/>
+<wire x1="32.00215625" y1="21.777" x2="38.07155625" y2="27.8464" width="1.5" layer="16"/>
+<wire x1="48.08" y1="27.406" x2="47.6396" y2="27.8464" width="1.5" layer="16"/>
+<wire x1="47.6396" y1="27.8464" x2="38.07155625" y2="27.8464" width="1.5" layer="16"/>
 </signal>
 <signal name="DRAIN1">
@@
 <wire x1="22.43" y1="19.43" x2="22.43" y2="24.067" width="1" layer="16"/>
 <wire x1="48.08" y1="23.44" x2="45.3377375" y2="23.44" width="2" layer="16"/>
-<wire x1="45.3377375" y1="23.44" x2="42.2813375" y2="26.4964" width="2" layer="16"/>
-<wire x1="42.2813375" y1="26.4964" x2="39.8655125" y2="26.4964" width="2" layer="16"/>
-<wire x1="39.8655125" y1="26.4964" x2="32.4437125" y2="19.0746" width="2" layer="16"/>
+<wire x1="45.3377375" y1="23.44" x2="42.6713375" y2="26.1064" width="1.5" layer="16"/>
+<wire x1="42.6713375" y1="26.1064" x2="39.4755125" y2="26.1064" width="1.5" layer="16"/>
+<wire x1="39.4755125" y1="26.1064" x2="32.4437125" y2="19.0746" width="1.5" layer="16"/>
 <wire x1="32.4437125" y1="19.0746" x2="26.4324" y2="19.0746" width="2" layer="16"/>
 <wire x1="26.4324" y1="19.0746" x2="22.43" y2="23.077" width="2" layer="16"/>
@@
 <contactref element="U$4" pad="2"/>
 <contactref element="U$5" pad="3"/>
-<wire x1="2.5" y1="35" x2="3" y2="35" width="1" layer="16"/>
-<wire x1="2.5" y1="35" x2="1.5336" y2="34.0336" width="1" layer="16"/>
+<wire x1="3" y1="35" x2="3" y2="34.98" width="1" layer="16"/>
+<wire x1="3" y1="34.98" x2="1.5336" y2="33.5136" width="1" layer="16"/>
 <wire x1="3" y1="2.46" x2="2.29" y2="2.46" width="1" layer="16"/>
 <wire x1="2.29" y1="2.46" x2="1.5936" y2="3.1564" width="1" layer="16"/>
 <wire x1="1.5936" y1="3.1564" x2="1.5936" y2="24.94" width="1" layer="16"/>
-<wire x1="1.5336" y1="25" x2="1.5336" y2="34.0336" width="1" layer="16"/>
+<wire x1="1.5336" y1="25" x2="1.5336" y2="33.5136" width="1" layer="16"/>
 <wire x1="9" y1="24.39" x2="2.1436" y2="24.39" width="1" layer="16"/>
 <wire x1="2.1436" y1="24.39" x2="1.5936" y2="24.94" width="1" layer="16"/>
 <wire x1="1.5936" y1="24.94" x2="1.5336" y2="25" width="1" layer="16"/>
 <wire x1="47.98895" y1="35" x2="48.54" y2="35" width="1" layer="16"/>
-<wire x1="4.43745" y1="36.4664" x2="3" y2="35.02895" width="1" layer="16"/>
-<wire x1="3" y1="35" x2="3" y2="35.02895" width="1" layer="16"/>
+<wire x1="4.49745" y1="36.4664" x2="3.03105" y2="35" width="1" layer="16"/>
+<wire x1="3" y1="35" x2="3.03105" y2="35" width="1" layer="16"/>
 <wire x1="46.52255" y1="36.4664" x2="47.98895" y2="35" width="1" layer="16"/>
-<wire x1="4.43745" y1="36.4664" x2="46.52255" y2="36.4664" width="1" layer="16"/>
+<wire x1="4.49745" y1="36.4664" x2="46.52255" y2="36.4664" width="1" layer="16"/>
 </signal>
 <signal name="5V">
 <contactref element="U$1" pad="5V_P"/>
 <polygon width="1.5" layer="1">
-<vertex x="56" y="41"/>
-<vertex x="56" y="-2"/>
+<vertex x="64" y="46"/>
+<vertex x="64" y="6"/>
 <vertex x="54" y="-4"/>
 <vertex x="-1" y="-4"/>
 <vertex x="-5" y="0"/>
 <vertex x="-5" y="36"/>
-<vertex x="0" y="41"/>
+<vertex x="5" y="46"/>
 </polygon>
 <contactref element="U$1" pad="5V1_P"/>
@@
 <wire x1="11.76" y1="14.23" x2="9" y2="14.23" width="1" layer="16"/>
 <contactref element="U$2" pad="2"/>
-<wire x1="17.53745" y1="33.3064" x2="20.82255" y2="33.3064" width="1" layer="1"/>
-<wire x1="16.7936" y1="32.56255" x2="17.53745" y2="33.3064" width="1" layer="1"/>
+<wire x1="17.86745" y1="33.3064" x2="20.82255" y2="33.3064" width="1" layer="1"/>
+<wire x1="16.7936" y1="32.23255" x2="17.86745" y2="33.3064" width="1" layer="1"/>
 <wire x1="21.24" y1="31.9" x2="21.24" y2="32.88895" width="1" layer="1"/>
 <wire x1="21.24" y1="32.88895" x2="20.82255" y2="33.3064" width="1" layer="1"/>
-<wire x1="16.7936" y1="18.4836" x2="16.7936" y2="32.56255" width="1" layer="1"/>
+<wire x1="16.7936" y1="18.4836" x2="16.7936" y2="32.23255" width="1" layer="1"/>
 </signal>
 <signal name="CANL">
@@
 <contactref element="U$4" pad="4"/>
 <contactref element="U$5" pad="1"/>
-<wire x1="43.1046" y1="35.81" x2="13.02" y2="35.81" width="0.5" layer="1"/>
-<wire x1="13.02" y1="35.81" x2="6.01" y2="28.8" width="0.5" layer="1"/>
-<wire x1="6.01" y1="28.8" x2="3.45" y2="28.8" width="0.5" layer="1"/>
+<wire x1="43.1046" y1="35.81" x2="16.88" y2="35.81" width="0.5" layer="1"/>
+<wire x1="16.88" y1="35.81" x2="9.87" y2="28.8" width="0.5" layer="1"/>
+<wire x1="9.87" y1="28.8" x2="3.45" y2="28.8" width="0.5" layer="1"/>
 <wire x1="3.45" y1="28.8" x2="3" y2="29.25" width="0.5" layer="1"/>
 <wire x1="3" y1="29.25" x2="3" y2="32.46" width="0.5" layer="1"/>
-<wire x1="3" y1="5" x2="3" y2="12" width="0.5" layer="1"/>
-<wire x1="3" y1="12" x2="3" y2="32.46" width="0.5" layer="1"/>
-<wire x1="9" y1="11.69" x2="3.31" y2="11.69" width="0.5" layer="1"/>
-<wire x1="3.31" y1="11.69" x2="3" y2="12" width="0.5" layer="1"/>
+<wire x1="3" y1="5" x2="3" y2="13.61" width="0.5" layer="1"/>
+<wire x1="3" y1="13.61" x2="3" y2="32.46" width="0.5" layer="1"/>
 <wire x1="47.2664" y1="33.7336" x2="48.54" y2="32.46" width="0.5" layer="1"/>
 <wire x1="43.1046" y1="35.81" x2="45.181" y2="33.7336" width="0.5" layer="1"/>
 <wire x1="45.181" y1="33.7336" x2="47.2664" y2="33.7336" width="0.5" layer="1"/>
+<wire x1="9" y1="11.69" x2="4.92" y2="11.69" width="0.5" layer="1"/>
+<wire x1="4.92" y1="11.69" x2="3" y2="13.61" width="0.5" layer="1"/>
 </signal>
 <signal name="CANH">
@@
 <contactref element="U$1" pad="SCK_P"/>
 <contactref element="U$2" pad="6"/>
-<wire x1="41" y1="9.15" x2="41" y2="9.25936875" width="1" layer="1"/>
-<wire x1="41" y1="9.25936875" x2="43.3464" y2="11.60576875" width="1" layer="1"/>
-<wire x1="43.3464" y1="11.60576875" x2="43.3464" y2="26.8336" width="1" layer="1"/>
-<wire x1="43.3464" y1="26.8336" x2="38.28" y2="31.9" width="1" layer="1"/>
-<wire x1="38.28" y1="31.9" x2="31.4" y2="31.9" width="1" layer="1"/>
+<wire x1="43.3464" y1="10.35576875" x2="42.14063125" y2="9.15" width="1" layer="1"/>
+<wire x1="41" y1="9.15" x2="42.14063125" y2="9.15" width="1" layer="1"/>
+<wire x1="43.3464" y1="10.35576875" x2="43.3464" y2="24.6236" width="1" layer="1"/>
+<wire x1="43.3464" y1="24.6236" x2="36.07" y2="31.9" width="1" layer="1"/>
+<wire x1="36.07" y1="31.9" x2="31.4" y2="31.9" width="1" layer="1"/>
 </signal>
 </signals>
