File: ACME - ACM Extention/PCB/ACME.brd (EAGLE design)
At the start: 49 x 34 mm, 17 parts, among them IC1 Optocoupler DIP, Q1 NGD8201ANT4G, Q2 NGD8201ANT4G

Commit message: ACME: ACME Ready for production
Parts:
- moved D1 0.75 mm to (27.3, 3.58)
- moved D0 0.09 mm to (14.8, 3.57)
Other:
- board text added: "MAX 30 VDC"
Changed lines of the file:
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@@
 <setting verticaltext="up"/>
 </settings>
-<grid distance="0.5" unitdist="mm" unit="mm" style="lines" multiple="1" display="yes" altdistance="0.01" altunitdist="mm" altunit="mm"/>
+<grid distance="0.5" unitdist="mm" unit="mm" style="lines" multiple="1" display="yes" altdistance="0.25" altunitdist="mm" altunit="mm"/>
 <layers>
 <layer number="1" name="Top" color="4" fill="1" visible="yes" active="yes"/>
@@
 <wire x1="0" y1="33" x2="0" y2="1" width="0" layer="20"/>
 <wire x1="0" y1="1" x2="1" y2="0" width="0" layer="20" curve="90"/>
-<text x="26.53" y="3.34" size="4" layer="25" distance="0" align="center">+</text>
+<text x="27.28" y="3.34" size="4" layer="25" distance="0" align="center">+</text>
 <text x="20.82" y="3.61" size="4" layer="25" distance="0" align="center">-</text>
-<text x="14.63" y="3.35" size="4" layer="25" distance="0" align="center">+</text>
+<text x="14.67" y="3.27" size="4" layer="25" distance="0" align="center">+</text>
 <text x="33.36" y="3.6" size="4" layer="25" distance="0" align="center">-</text>
 <text x="5.46" y="30.51" size="1" layer="25" align="center-right">12V</text>
@@
 <hole x="10.69" y="2.89" drill="2"/>
 <hole x="46" y="3" drill="3"/>
-<text x="17.64" y="3.02" size="1.778" layer="25" align="center">A</text>
-<text x="29.8" y="3.16" size="1.778" layer="25" align="center">B</text>
+<text x="17.77" y="1.145" size="1.778" layer="25" align="center">A</text>
+<text x="30.24" y="1.145" size="1.778" layer="25" align="center">B</text>
 <text x="21" y="32.5" size="1.778" layer="25" align="center">ACME - ACM Extention</text>
 <text x="42.01" y="1.49" size="1" layer="25" align="center">Rev. A</text>
@@
 <text x="2" y="18.5" size="1.1" layer="26" rot="MR270" align="center">*Designed by Humans from Earth*</text>
 <text x="19.5" y="31" size="1" layer="25" align="center-left">with dual mosfet switch</text>
-<wire x1="19.5" y1="30.5" x2="34" y2="30.5" width="0.1" layer="25"/>
+<wire x1="19.5" y1="30.5" x2="34.5" y2="30.5" width="0.1" layer="25"/>
 <hole x="35" y="20.5" drill="3"/>
 <dimension x1="10.5" y1="7" x2="7.5" y2="7" x3="9" y3="6.84" textsize="0.71" layer="22" width="0.03" precision="0" visible="yes"/>
@@
 </polygon>
 <hole x="2" y="2" drill="3"/>
+<rectangle x1="31.68" y1="-0.14" x2="34.88" y2="0.95" layer="26"/>
+<rectangle x1="19.02" y1="-0.3" x2="22.22" y2="0.89" layer="26"/>
+<text x="30.24" y="1.145" size="1.778" layer="26" rot="MR0" align="center">B</text>
+<text x="17.77" y="1.145" size="1.778" layer="26" rot="MR0" align="center">A</text>
+<text x="30.25" y="2" size="1" layer="26" rot="MR90" align="center-left">MAX
+30 VDC</text>
+<text x="17.75" y="2" size="1" layer="26" rot="MR90" align="center-left">MAX
+30 VDC</text>
 </plain>
 <attributes>
@@
 <attribute name="RS_PART_NUMBER" value="7470901" x="-3.86" y="-26.4435" size="1.778" layer="28" rot="MR0" display="off"/>
 <attribute name="RS_PRICE-STOCK" value="http://uk.rs-online.com/web/p/products/7470901" x="-3.86" y="-26.4435" size="1.778" layer="28" rot="MR0" display="off"/>
-<attribute name="VALUE" x="44.4" y="-2.3135" size="1.27" layer="28" rot="MR0" align="center"/>
+<attribute name="VALUE" x="12.4" y="-5.3135" size="1.27" layer="28" rot="MR0" align="center"/>
 </element>
 <element name="Q2" library="NGD8201ANT4G_Mosfet" package="TO229P990X238-4N" value="NGD8201ANT4G" x="29.037" y="10.3765" smashed="yes" rot="MR0">
@@
 <attribute name="RS_PART_NUMBER" value="7470901" x="-6.523" y="-26.4535" size="1.778" layer="28" rot="MR0" display="off"/>
 <attribute name="RS_PRICE-STOCK" value="http://uk.rs-online.com/web/p/products/7470901" x="-6.523" y="-26.4535" size="1.778" layer="28" rot="MR0" display="off"/>
-<attribute name="VALUE" x="32.15" y="10.5735" size="1.27" layer="28" rot="MR90" align="center"/>
+<attribute name="VALUE" x="31.4265" y="-5.35" size="1.27" layer="28" rot="MR0" align="center"/>
 </element>
 <element name="R1" library="ERA-3AEB2262V(0603 Resistor)" package="RESC1608X55N" value="" x="33.86" y="10.3765" smashed="yes" rot="MR270">
@@
 <attribute name="RS_PRICE-STOCK" value="" x="25.19" y="15.08" size="1.778" layer="28" rot="MR180" display="off"/>
 </element>
-<element name="D0" library="wirepad" library_urn="urn:adsk.eagle:library:412" package="5-2,5" package3d_urn="urn:adsk.eagle:package:30845/1" value="" x="14.71" y="3.65" smashed="yes" rot="MR180">
-<attribute name="NAME" x="16.44" y="1.342" size="1.27" layer="26" ratio="10" rot="MR180"/>
-<attribute name="VALUE" x="14.61" y="0.85" size="0.0254" layer="28" rot="MR180"/>
+<element name="D0" library="wirepad" library_urn="urn:adsk.eagle:library:412" package="5-2,5" package3d_urn="urn:adsk.eagle:package:30845/1" value="" x="14.75" y="3.57" smashed="yes" rot="MR180">
+<attribute name="NAME" x="13.98" y="-1.738" size="1.27" layer="26" ratio="10" rot="MR180"/>
+<attribute name="VALUE" x="14.65" y="0.77" size="0.0254" layer="28" rot="MR180"/>
 </element>
 <element name="S0" library="wirepad" library_urn="urn:adsk.eagle:library:412" package="5-2,5" package3d_urn="urn:adsk.eagle:package:30845/1" value="" x="20.621" y="3.65" smashed="yes" rot="MR0">
-<attribute name="NAME" x="22.279" y="1.484" size="1.27" layer="26" ratio="10" rot="MR180"/>
+<attribute name="NAME" x="19.779" y="-1.516" size="1.27" layer="26" ratio="10" rot="MR180"/>
 <attribute name="VALUE" x="20.721" y="6.45" size="0.0254" layer="28" rot="MR0"/>
 </element>
 <element name="S1" library="wirepad" library_urn="urn:adsk.eagle:library:412" package="5-2,5" package3d_urn="urn:adsk.eagle:package:30845/1" value="" x="33.276" y="3.73" smashed="yes" rot="MR180">
-<attribute name="NAME" x="35.01" y="1.628" size="1.27" layer="26" ratio="10" rot="MR180"/>
+<attribute name="NAME" x="32.01" y="-1.372" size="1.27" layer="26" ratio="10" rot="MR180"/>
 <attribute name="VALUE" x="33.176" y="0.93" size="0.0254" layer="28" rot="MR180"/>
 </element>
-<element name="D1" library="wirepad" library_urn="urn:adsk.eagle:library:412" package="5-2,5" package3d_urn="urn:adsk.eagle:package:30845/1" value="" x="26.51" y="3.58" smashed="yes" rot="MR180">
-<attribute name="NAME" x="28.14" y="1.382" size="1.27" layer="26" ratio="10" rot="MR180"/>
-<attribute name="VALUE" x="26.41" y="0.78" size="0.0254" layer="28" rot="MR180"/>
+<element name="D1" library="wirepad" library_urn="urn:adsk.eagle:library:412" package="5-2,5" package3d_urn="urn:adsk.eagle:package:30845/1" value="" x="27.26" y="3.58" smashed="yes" rot="MR180">
+<attribute name="NAME" x="26.89" y="-2.118" size="1.27" layer="26" ratio="10" rot="MR180" align="center"/>
+<attribute name="VALUE" x="27.16" y="0.78" size="0.0254" layer="28" rot="MR180"/>
 </element>
 <element name="U$1" library="ACM_Pindown" package="ACM_CAS_FP" value="ACM_CASTELLATED" x="6.69" y="-0.11" smashed="yes"/>
@@
 <wire x1="15.25" y1="16.3" x2="14.51" y2="16.3" width="0.85" layer="16"/>
 <wire x1="14.51" y1="16.3" x2="11.86" y2="13.65" width="0.85" layer="16"/>
-<wire x1="14.71" y1="3.65" x2="14.71" y2="9.5365" width="2.54" layer="16"/>
-<wire x1="14.71" y1="9.5365" x2="13.86" y2="10.3865" width="2.54" layer="16"/>
+<wire x1="14.75" y1="3.57" x2="14.75" y2="9.4965" width="2.54" layer="16"/>
+<wire x1="14.75" y1="9.4965" x2="13.86" y2="10.3865" width="2.54" layer="16"/>
 <wire x1="11.86" y1="13.65" x2="11.86" y2="12.3865" width="0.85" layer="16"/>
 <wire x1="11.86" y1="12.3865" x2="13.86" y2="10.3865" width="0.85" layer="16"/>
@@
 <wire x1="26.61" y1="14.46" x2="26.61" y2="10.5495" width="0.85" layer="16"/>
 <wire x1="26.61" y1="10.5495" x2="26.437" y2="10.3765" width="0.85" layer="16"/>
-<wire x1="26.51" y1="3.58" x2="26.51" y2="10.3035" width="2.54" layer="16"/>
-<wire x1="26.51" y1="10.3035" x2="26.437" y2="10.3765" width="2.54" layer="16"/>
+<wire x1="27.26" y1="3.58" x2="27.26" y2="9.5535" width="2.54" layer="16"/>
+<wire x1="27.26" y1="9.5535" x2="26.437" y2="10.3765" width="2.54" layer="16"/>
 </signal>
 <signal name="N$2">
@@
 </drawing>
 <compatibility>
+<note version="6.3" minversion="6.2.2" severity="warning">
+Since Version 6.2.2 text objects can contain more than one line,
+which will not be processed correctly with this version.
+</note>
 <note version="8.2" severity="warning">
 Since Version 8.2, EAGLE supports online libraries. The ids
